File: Busboard.kicad_pcb (KiCad board)
At the start: 2 copper layers, 400 x 45 mm, 50 parts, among them J1 Conn_01x02, J10 Conn_02x08_Counter_Clockwise, J11 Conn_02x08_Counter_Clockwise, J12 Conn_01x02, J13 Conn_01x02, J14 Conn_01x02, J15 Conn_01x02, J16 Conn_02x08_Counter_Clockwise, J17 Conn_02x08_Counter_Clockwise, J18 Conn_02x08_Counter_Clockwise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

Commit message: fix
Parts:
- removed the REF** at (264.0, 270.0)
- removed the REF** at (264.0, 305.0)
- removed the REF** at (305.5, 270.0)
- removed the REF** at (305.5, 305.0)
- removed the REF** at (133.5, 270.0)
- removed the REF** at (90.0, 270.0)
- removed the REF** at (177.0, 270.0)
- removed the REF** at (220.5, 305.0)
- removed the REF** at (220.5, 270.0)
- added REF**: MountingHole_3.2mm_M3-No-cu, own_libraries:MountingHole_3.2mm_M3-No-cu, F.Cu at (264.0, 269.6)
- added REF**: MountingHole_3.2mm_M3-No-cu, own_libraries:MountingHole_3.2mm_M3-No-cu, F.Cu at (264.0, 305.4)
- added REF**: MountingHole_3.2mm_M3-No-cu, own_libraries:MountingHole_3.2mm_M3-No-cu, F.Cu at (305.5, 269.6)
- added REF**: MountingHole_3.2mm_M3-No-cu, own_libraries:MountingHole_3.2mm_M3-No-cu, F.Cu at (305.5, 305.4)
- added REF**: MountingHole_3.2mm_M3-No-cu, own_libraries:MountingHole_3.2mm_M3-No-cu, F.Cu at (133.5, 269.6)
- added REF**: MountingHole_3.2mm_M3-No-cu, own_libraries:MountingHole_3.2mm_M3-No-cu, F.Cu at (89.6, 269.6)
- added REF**: MountingHole_3.2mm_M3-No-cu, own_libraries:MountingHole_3.2mm_M3-No-cu, F.Cu at (177.0, 269.6)
- added REF**: MountingHole_3.2mm_M3-No-cu, own_libraries:MountingHole_3.2mm_M3-No-cu, F.Cu at (220.5, 305.4)
- added REF**: MountingHole_3.2mm_M3-No-cu, own_libraries:MountingHole_3.2mm_M3-No-cu, F.Cu at (220.5, 269.6)
- moved REF** 0.57 mm to (89.6, 305.4)
- moved REF** 0.57 mm to (480.4, 269.6)
- moved REF** 0.57 mm to (480.4, 305.4)
- moved REF** 0.40 mm to (133.5, 305.4)
- moved REF** 0.40 mm to (392.8, 305.4)
- moved REF** 0.40 mm to (349.1, 269.6)
- moved REF** 0.40 mm to (349.1, 305.4)
- moved REF** 0.40 mm to (177.0, 305.4)
- moved REF** 0.40 mm to (436.4, 269.6)
- moved REF** 0.40 mm to (436.4, 305.4)
- moved REF** 0.40 mm to (392.8, 269.6)
Changed lines of the file:
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@@
   )
   (setup
-    (last_trace_width 0.254)
+    (last_trace_width 0.25)
     (user_trace_width 0.254)
     (trace_clearance 0.2)
@@
     (via_min_size 0.4)
     (via_min_drill 0.3)
-    (uvia_size 0.3)
-    (uvia_drill 0.1)
+    (uvia_size 0.8)
+    (uvia_drill 0.4)
     (uvias_allowed no)
-    (uvia_min_size 0.2)
+    (uvia_min_size 0.4)
     (uvia_min_drill 0.1)
     (edge_width 0.05)
@@
     (via_dia 0.8)
     (via_drill 0.4)
-    (uvia_dia 0.3)
-    (uvia_drill 0.1)
+    (uvia_dia 0.8)
+    (uvia_drill 0.4)
     (add_net +12V)
     (add_net -12V)
@@
   )
   (module own_libraries:MountingHole_3.2mm_M3-No-cu (layer F.Cu)
-    (at 133.5 305)
+    (at 133.5 305.4)
     (descr "Mounting Hole 3.2mm, no annular, M3")
     (tags "mounting hole 3.2mm no annular m3")
@@
   )
   (module own_libraries:MountingHole_3.2mm_M3-No-cu (layer F.Cu)
-    (at 133.5 270)
+    (at 133.5 269.6)
     (descr "Mounting Hole 3.2mm, no annular, M3")
     (tags "mounting hole 3.2mm no annular m3")
@@
   )
   (module own_libraries:MountingHole_3.2mm_M3-No-cu (layer F.Cu)
-    (at 177 305)
+    (at 177 305.4)
     (descr "Mounting Hole 3.2mm, no annular, M3")
     (tags "mounting hole 3.2mm no annular m3")
@@
   )
   (module own_libraries:MountingHole_3.2mm_M3-No-cu (layer F.Cu)
-    (at 177 270)
+    (at 177 269.6)
     (descr "Mounting Hole 3.2mm, no annular, M3")
     (tags "mounting hole 3.2mm no annular m3")
@@
   )
   (module own_libraries:MountingHole_3.2mm_M3-No-cu (layer F.Cu)
-    (at 220.5 305)
+    (at 220.5 305.4)
     (descr "Mounting Hole 3.2mm, no annular, M3")
     (tags "mounting hole 3.2mm no annular m3")
@@
   )
   (module own_libraries:MountingHole_3.2mm_M3-No-cu (layer F.Cu)
-    (at 220.5 270)
+    (at 220.5 269.6)
     (descr "Mounting Hole 3.2mm, no annular, M3")
     (tags "mounting hole 3.2mm no annular m3")
@@
   )
   (module own_libraries:MountingHole_3.2mm_M3-No-cu (layer F.Cu)
-    (at 436.375 270)
+    (at 436.375 269.6)
     (descr "Mounting Hole 3.2mm, no annular, M3")
     (tags "mounting hole 3.2mm no annular m3")
@@
   )
   (module own_libraries:MountingHole_3.2mm_M3-No-cu (layer F.Cu)
-    (at 436.375 305)
+    (at 436.375 305.4)
     (descr "Mounting Hole 3.2mm, no annular, M3")
     (tags "mounting hole 3.2mm no annular m3")
@@
   )
   (module own_libraries:MountingHole_3.2mm_M3-No-cu (layer F.Cu)
-    (at 392.75 270)
+    (at 392.75 269.6)
     (descr "Mounting Hole 3.2mm, no annular, M3")
     (tags "mounting hole 3.2mm no annular m3")
@@
   )
   (module own_libraries:MountingHole_3.2mm_M3-No-cu (layer F.Cu)
-    (at 392.75 305)
+    (at 392.75 305.4)
     (descr "Mounting Hole 3.2mm, no annular, M3")
     (tags "mounting hole 3.2mm no annular m3")
@@
   )
   (module own_libraries:MountingHole_3.2mm_M3-No-cu (layer F.Cu)
-    (at 349.125 270)
+    (at 349.125 269.6)
     (descr "Mounting Hole 3.2mm, no annular, M3")
     (tags "mounting hole 3.2mm no annular m3")
@@
   )
   (module own_libraries:MountingHole_3.2mm_M3-No-cu (layer F.Cu)
-    (at 349.125 305)
+    (at 349.125 305.4)
     (descr "Mounting Hole 3.2mm, no annular, M3")
     (tags "mounting hole 3.2mm no annular m3")
@@
   )
   (module own_libraries:MountingHole_3.2mm_M3-No-cu (layer F.Cu)
-    (at 264 270)
+    (at 264 269.6)
     (descr "Mounting Hole 3.2mm, no annular, M3")
     (tags "mounting hole 3.2mm no annular m3")
@@
   )
   (module own_libraries:MountingHole_3.2mm_M3-No-cu (layer F.Cu)
-    (at 264 305)
+    (at 264 305.4)
     (descr "Mounting Hole 3.2mm, no annular, M3")
     (tags "mounting hole 3.2mm no annular m3")
@@
   )
   (module own_libraries:MountingHole_3.2mm_M3-No-cu (layer F.Cu)
-    (at 305.5 270)
+    (at 305.5 269.6)
     (descr "Mounting Hole 3.2mm, no annular, M3")
     (tags "mounting hole 3.2mm no annular m3")
@@
   )
   (module own_libraries:MountingHole_3.2mm_M3-No-cu (layer F.Cu)
-    (at 305.5 305)
+    (at 305.5 305.4)
     (descr "Mounting Hole 3.2mm, no annular, M3")
     (tags "mounting hole 3.2mm no annular m3")
@@
   )
   (module own_libraries:MountingHole_3.2mm_M3-No-cu (layer F.Cu)
-    (at 480 270)
+    (at 480.4 269.6)
     (descr "Mounting Hole 3.2mm, no annular, M3")
     (tags "mounting hole 3.2mm no annular m3")
@@
   )
   (module own_libraries:MountingHole_3.2mm_M3-No-cu (layer F.Cu)
-    (at 480 305)
+    (at 480.4 305.4)
     (descr "Mounting Hole 3.2mm, no annular, M3")
     (tags "mounting hole 3.2mm no annular m3")
@@
   )
   (module own_libraries:MountingHole_3.2mm_M3-No-cu (layer F.Cu)
-    (at 90 305)
+    (at 89.6 305.4)
     (descr "Mounting Hole 3.2mm, no annular, M3")
     (tags "mounting hole 3.2mm no annular m3")
@@
   )
   (module own_libraries:MountingHole_3.2mm_M3-No-cu (layer F.Cu)
-    (at 90 270)
+    (at 89.6 269.6)
     (descr "Mounting Hole 3.2mm, no annular, M3")
     (tags "mounting hole 3.2mm no annular m3")
@@
     (polygon
       (pts
-        (xy 84.5 295.5) (xy 84.5 310.5) (xy 485.5 310.5) (xy 485.5 295.5)
+        (xy 84.6 295.6) (xy 84.5 310.5) (xy 485.5 310.5) (xy 485.5 295.6)
       )
     )
@@
     (polygon
       (pts
-        (xy 103 287) (xy 266.5 287) (xy 266.5 281) (xy 308 281) (xy 308 287)
-        (xy 467 287) (xy 467 279) (xy 485.5 279) (xy 485.5 264.5) (xy 84.5 264.5)
-        (xy 84.5 279) (xy 103 279)
-      )
-    )
-  )
-  (zone (net 1) (net_name +12V) (layer B.Cu) (hatch edge 0.508)
-    (connect_pads (clearance 0.508))
-    (min_thickness 0.254)
-    (fill yes (arc_segments 32) (thermal_gap 0.508) (thermal_bridge_width 1.016))
-    (polygon
-      (pts
-        (xy 103 287) (xy 266.5 287) (xy 266.5 281) (xy 308 281) (xy 308 287)
-        (xy 467 287) (xy 467 279) (xy 485.5 279) (xy 485.5 264.5) (xy 84.5 264.5)
-        (xy 84.5 279) (xy 103 279)
+        (xy 103.1 286.9) (xy 266.4 286.9) (xy 266.4 280.9) (xy 308.1 280.9) (xy 308.1 286.9)
+        (xy 466.9 286.9) (xy 466.9 278.9) (xy 485.5 278.9) (xy 485.5 264.5) (xy 84.5 264.5)
+        (xy 84.5 278.9) (xy 103.1 278.9)
       )
     )
@@
     (polygon
       (pts
-        (xy 84.5 295.5) (xy 84.5 310.5) (xy 485.5 310.5) (xy 485.5 295.5)
+        (xy 84.5 295.6) (xy 84.5 310.5) (xy 485.5 310.5) (xy 485.4 295.6)
       )
     )
+  )
+  (zone (net 1) (net_name +12V) (layer B.Cu) (hatch edge 0.508)
+    (connect_pads (clearance 0.508))
+    (min_thickness 0.254)
+    (fill yes (arc_segments 32) (thermal_gap 0.508) (thermal_bridge_width 1.016))
+    (polygon
+      (pts
+        (xy 103.1 286.9) (xy 266.4 286.9) (xy 266.4 280.9) (xy 308.1 280.9) (xy 308.1 286.9)
+        (xy 466.9 286.9) (xy 466.9 278.9) (xy 485.5 278.9) (xy 485.5 264.5) (xy 84.5 264.5)
+        (xy 84.5 278.9) (xy 103.1 278.9)
+      )
+    )

Commit message: v02
OK, I added 5V and gate and CV. No regulator or jumpers, though.
Parts:
- added J27: Conn_01x02, own_libraries:FASTON_6.35_mm, F.Cu at (280.5, 276.0)
- moved J12 4.50 mm to (289.5, 276.0)
- moved D2 2.53 mm to (301.4, 298.2)
- moved R2 2.53 mm to (296.4, 297.2)
- moved D1 2.41 mm to (301.4, 282.8)
- moved R1 2.41 mm to (296.4, 281.3)
- moved J13 0.50 mm to (280.5, 289.0)
- moved J14 0.50 mm to (289.5, 289.0)
Connections:
- J10 pad 1: Net-(J10-Pad1) -> Gate
- J10 pad 2: Net-(J10-Pad2) -> Gate
- J10 pad 3: Net-(J10-Pad3) -> CV
- J10 pad 4: Net-(J10-Pad4) -> CV
- J10 pad 5: Net-(J10-Pad5) -> +5V
- J10 pad 6: Net-(J10-Pad6) -> +5V
- J11 pad 1: Net-(J11-Pad1) -> Gate
- J11 pad 2: Net-(J11-Pad2) -> Gate
- J11 pad 3: Net-(J11-Pad3) -> CV
- J11 pad 4: Net-(J11-Pad4) -> CV
- J11 pad 5: Net-(J11-Pad5) -> +5V
- J11 pad 6: Net-(J11-Pad6) -> +5V
- J16 pad 1: Net-(J16-Pad1) -> Gate
- J16 pad 2: Net-(J16-Pad2) -> Gate
- J16 pad 3: Net-(J16-Pad3) -> CV
- J16 pad 4: Net-(J16-Pad4) -> CV
- J16 pad 5: Net-(J16-Pad5) -> +5V
- J16 pad 6: Net-(J16-Pad6) -> +5V
- J17 pad 1: Net-(J17-Pad1) -> Gate
- J17 pad 2: Net-(J17-Pad2) -> Gate
- J17 pad 3: Net-(J17-Pad3) -> CV
- J17 pad 4: Net-(J17-Pad4) -> CV
- J17 pad 5: Net-(J17-Pad5) -> +5V
- J17 pad 6: Net-(J17-Pad6) -> +5V
- J18 pad 1: Net-(J18-Pad1) -> Gate
- J18 pad 2: Net-(J18-Pad2) -> Gate
- J18 pad 3: Net-(J18-Pad3) -> CV
- J18 pad 4: Net-(J18-Pad4) -> CV
- J18 pad 5: Net-(J18-Pad5) -> +5V
- J18 pad 6: Net-(J18-Pad6) -> +5V
- J19 pad 1: Net-(J19-Pad1) -> Gate
- J19 pad 2: Net-(J19-Pad2) -> Gate
- J19 pad 3: Net-(J19-Pad3) -> CV
- J19 pad 4: Net-(J19-Pad4) -> CV
- J19 pad 5: Net-(J19-Pad5) -> +5V
- J19 pad 6: Net-(J19-Pad6) -> +5V
- J20 pad 1: Net-(J20-Pad1) -> Gate
- J20 pad 2: Net-(J20-Pad2) -> Gate
- J20 pad 3: Net-(J20-Pad3) -> CV
- J20 pad 4: Net-(J20-Pad4) -> CV
- J20 pad 5: Net-(J20-Pad5) -> +5V
- J20 pad 6: Net-(J20-Pad6) -> +5V
- J21 pad 1: Net-(J21-Pad1) -> Gate
- J21 pad 2: Net-(J21-Pad2) -> Gate
- J21 pad 3: Net-(J21-Pad3) -> CV
- J21 pad 4: Net-(J21-Pad4) -> CV
- J21 pad 5: Net-(J21-Pad5) -> +5V
- J21 pad 6: Net-(J21-Pad6) -> +5V
- J22 pad 1: Net-(J22-Pad1) -> Gate
- J22 pad 2: Net-(J22-Pad2) -> Gate
- J22 pad 3: Net-(J22-Pad3) -> CV
- J22 pad 4: Net-(J22-Pad4) -> CV
- J22 pad 5: Net-(J22-Pad5) -> +5V
- J22 pad 6: Net-(J22-Pad6) -> +5V
- J5 pad 1: Net-(J5-Pad1) -> Gate
- J5 pad 2: Net-(J5-Pad2) -> Gate
- J5 pad 3: Net-(J5-Pad3) -> CV
- J5 pad 4: Net-(J5-Pad4) -> CV
- J5 pad 5: Net-(J5-Pad5) -> +5V
- J5 pad 6: Net-(J5-Pad6) -> +5V
- J6 pad 1: Net-(J6-Pad1) -> Gate
- J6 pad 2: Net-(J6-Pad2) -> Gate
- J6 pad 3: Net-(J6-Pad3) -> CV
- J6 pad 4: Net-(J6-Pad4) -> CV
- J6 pad 5: Net-(J6-Pad5) -> +5V
- J6 pad 6: Net-(J6-Pad6) -> +5V
- J7 pad 1: Net-(J7-Pad1) -> Gate
- J7 pad 2: Net-(J7-Pad2) -> Gate
- J7 pad 3: Net-(J7-Pad3) -> CV
- J7 pad 4: Net-(J7-Pad4) -> CV
- J7 pad 5: Net-(J7-Pad5) -> +5V
- J7 pad 6: Net-(J7-Pad6) -> +5V
- J8 pad 1: Net-(J8-Pad1) -> Gate
- J8 pad 2: Net-(J8-Pad2) -> Gate
- J8 pad 3: Net-(J8-Pad3) -> CV
- J8 pad 4: Net-(J8-Pad4) -> CV
- J8 pad 5: Net-(J8-Pad5) -> +5V
- J8 pad 6: Net-(J8-Pad6) -> +5V
- J9 pad 1: Net-(J9-Pad1) -> Gate
- J9 pad 2: Net-(J9-Pad2) -> Gate
- J9 pad 3: Net-(J9-Pad3) -> CV
- J9 pad 4: Net-(J9-Pad4) -> CV
- J9 pad 5: Net-(J9-Pad5) -> +5V
- J9 pad 6: Net-(J9-Pad6) -> +5V
Routing:
- net Gate: track 0.00 -> 370.2 mm
- net CV: track 0.00 -> 367.0 mm
- net +5V: track 0.00 -> 365.2 mm
- net GND: track 1.96 -> 4.26 mm
Other:
- board text added: "+5V"
- board text removed: "No 5V - No CV - No Gate!"

Commit message: v02
Added jumpers for Gate and CV.
Changed to screw terminals.
Parts:
- removed J13, J14, J15, J23, J24, J25, J26, J27: Conn_01x02, own_libraries:FASTON_6.35_mm
- J1, J2, J3: value Conn_01x02 -> Screw_Terminal_01x05; footprint own_libraries:FASTON_6.35_mm -> TerminalBlock_RND:TerminalBlock_RND_205-00048_1x05_P5.00mm_Horizontal
- J12, J4: value Conn_01x02 -> Conn_01x02_Male; footprint own_libraries:FASTON_6.35_mm -> Connector_PinHeader_2.54mm:PinHeader_1x02_P2.54mm_Vertical
- moved J1 375.5 mm to (471.6, 297.4), turned to 90 degrees
- moved J2 188.1 mm to (285.0, 278.4), turned to 270 degrees
- moved J4 179.7 mm to (275.0, 275.8), turned to 270 degrees
- moved J3 13.4 mm to (97.8, 277.6), turned to 270 degrees
- moved J12 7.90 mm to (297.4, 276.0), turned to 270 degrees
- moved D1 3.00 mm to (301.4, 285.8)
- moved R1 1.91 mm to (296.6, 283.2), turned to 180 degrees
- moved D2 1.00 mm to (301.4, 297.2)
- turned R2 to 180 degrees
Connections:
- J1 pad 1: +12V -> -12V
- J1 pad 2: +12V -> GND
- J10 pad 1: Gate -> Net-(J10-Pad1)
- J10 pad 2: Gate -> Net-(J10-Pad1)
- J10 pad 3: CV -> Net-(J10-Pad3)
- J10 pad 4: CV -> Net-(J10-Pad3)
- J12 pad 1: +12V -> CV
- J12 pad 2: +12V -> Net-(J10-Pad3)
- J16 pad 1: Gate -> Net-(J10-Pad1)
- J16 pad 2: Gate -> Net-(J10-Pad1)
- J16 pad 3: CV -> Net-(J10-Pad3)
- J16 pad 4: CV -> Net-(J10-Pad3)
- J2 pad 1: GND -> +5V
- J2 pad 2: GND -> +12V
- J3 pad 1: GND -> +5V
- J3 pad 2: GND -> +12V
- J4 pad 1: -12V -> Gate
- J4 pad 2: -12V -> Net-(J10-Pad1)
- J5 pad 1: Gate -> Net-(J10-Pad1)
- J5 pad 2: Gate -> Net-(J10-Pad1)
- J5 pad 3: CV -> Net-(J10-Pad3)
- J5 pad 4: CV -> Net-(J10-Pad3)
- J6 pad 1: Gate -> Net-(J10-Pad1)
- J6 pad 2: Gate -> Net-(J10-Pad1)
- J6 pad 3: CV -> Net-(J10-Pad3)
- J6 pad 4: CV -> Net-(J10-Pad3)
- J7 pad 1: Gate -> Net-(J10-Pad1)
- J7 pad 2: Gate -> Net-(J10-Pad1)
- J7 pad 3: CV -> Net-(J10-Pad3)
- J7 pad 4: CV -> Net-(J10-Pad3)
- J8 pad 1: Gate -> Net-(J10-Pad1)
- J8 pad 2: Gate -> Net-(J10-Pad1)
- J8 pad 3: CV -> Net-(J10-Pad3)
- J8 pad 4: CV -> Net-(J10-Pad3)
- J9 pad 1: Gate -> Net-(J10-Pad1)
- J9 pad 2: Gate -> Net-(J10-Pad1)
- J9 pad 3: CV -> Net-(J10-Pad3)
- J9 pad 4: CV -> Net-(J10-Pad3)
Routing:
- net CV: track 367.0 -> 166.2 mm, vias 0 -> 1
- net Net-(J10-Pad3): track 0.00 -> 194.9 mm, vias 0 -> 1
- net Gate: track 370.2 -> 194.4 mm
- net Net-(J10-Pad1): track 0.00 -> 167.6 mm
- net +5V: track 365.2 -> 383.2 mm
- net Net-(D1-Pad2): track 5.86 -> 3.88 mm
- net GND: track 4.26 -> 2.46 mm, vias 0 -> 22
- net Net-(D2-Pad1): track 5.01 -> 4.01 mm
- net -12V: vias 0 -> 20
- net +12V: vias 0 -> 34
Other:
- board text added: "5V"
- board text added: "CV"
- board text added: "Eurorack Busboard v02 cc-by-sa-3.0"
- board text added: "Gate"
- board text removed: "+5V"
